Commit message: add lwr with ati sensor

File: examples/resources/lwr.urdf (robot description, URDF)
Before this commit: robot lwr, 11 links, 10 joints
Links:
- added link ati_base_link, mass 0.521; collision mesh filename=package://lwr_description/meshes/ati_sensor/ati_sensor_coll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; visual mesh filename=package://lwr_description/meshes/ati_sensor/ati_sensor.stl
- added link ati_link, mass 0.001; collision cylinder length=0.01 radius=0.03; visual cylinder length=0.01 radius=0.03
- link base_link: geometry 
Joints:
- added joint ati_base_joint: type fixed, parent link_7, child ati_base_link, origin xyz=0 0 0.045 rpy=0 0 0.349065850399, limit lower=0 upper=0 effort=400 velocity=0
- added joint ati_joint: type fixed, parent ati_base_link, child ati_link, origin xyz=0 0 0.0036 rpy=0 0 0, limit lower=0 upper=0 effort=400 velocity=0
- joint world_joint: limit lower=0 upper=0 effort=400000 velocity=0 -> (none)
