Commit message: Added urdf from panda robot Need to verify the inertial properties

File: examples/resources/panda.urdf (robot description, URDF)
Before this commit: robot panda, 10 links, 9 joints
Links:
- link panda_link0: mass 1.2 -> 2.0
- link panda_link1: mass 2.0 -> 2.7
- link panda_link2: mass 2.0 -> 2.7
- link panda_link3: mass 2.0 -> 2.7
- link panda_link4: mass 2.0 -> 2.7
- link panda_link5: mass 2.0 -> 1.7
- link panda_link6: mass 1.0 -> 1.6
- link panda_link7: mass 0.2 -> 1
Joints:
- joint panda_joint4: limit lower=-3.0718 upper=-0.0698 effort=87 velocity=2.1750 -> lower=-3.0718 upper=3.0718 effort=87 velocity=2.1750
- joint panda_joint6: limit lower=-0.0175 upper=3.7525 effort=12 velocity=2.6100 -> lower=-3.7525 upper=3.7525 effort=12 velocity=2.6100
